File: fpga2.kicad_sch (KiCad schematic)
At the start: 6 parts, among them U1 XC6SLX25-FTG256, X1 50 MHz

Commit message: Updated revA: replaced resistors with IC for HDMI protection
Parts:
- renumbered C67 to C37, R9 to R12, R12 to R13, R11 to R14, U1 to U7

Commit message: Cleanup revA
Connections:
- net TP1 renamed UBUS_6
- net TP2 renamed UBUS_0
- net TP3 renamed UBUS_3
- net TP4 renamed UBUS_2
- net TP5 renamed UBUS_1
- net TP6 renamed UBUS_9
- net WA0 renamed UBUS_8
- net WA1: no longer names the net of U7.P8 (IO_L30P_GCLK1_D13_2)
- net WA2: no longer names the net of U7.N8 (IO_L29N_GCLK2_2)
- net WD0: no longer names the net of U7.R9 (IO_L23P_2)
- net WD1 renamed UBUS_10
- net WD11: no longer names the net of U7.M4 (IO_L1P_3)
- net WD15: no longer names the net of U7.N6 (IO_L64N_D9_2)
- net WD3: no longer names the net of U7.M5 (IO_L2P_3)
- net WD6: no longer names the net of U7.N5 (IO_L49P_D3_2)
- net WD7: no longer names the net of U7.T5 (IO_L48N_RDWR_B_VREF_2)
- net WD8 renamed UBUS_4
- net ~{WCS0}: no longer names the net of U7.P6 (IO_L47P_2)
- net ~{WRD}: no longer names the net of U7.P7 (IO_L31P_GCLK31_D14_2)
- net ~{WWR}: no longer names the net of U7.R7 (IO_L32P_GCLK29_2)
- no-connect marks 1 -> 12

Commit message: Updated revB
Parts:
- added C86: 100n, Capacitor_SMD:C_0603_1608Metric_Pad1.08x0.95mm_HandSolder, symbol Device:C
- added JP1: Flashboot, Jumper:SolderJumper-2_P1.3mm_Open_RoundedPad1.0x1.5mm, symbol Jumper:Jumper_2_Open
- added R20: 10k, Resistor_SMD:R_0603_1608Metric_Pad0.98x0.95mm_HandSolder, symbol Device:R
- added TP1: TDI, TestPoint:TestPoint_Pad_D1.0mm, symbol Connector:TestPoint
- added TP2: TDO, TestPoint:TestPoint_Pad_D1.0mm, symbol Connector:TestPoint
- added TP3: TMS, TestPoint:TestPoint_Pad_D1.0mm, symbol Connector:TestPoint
- added TP4: TCK, TestPoint:TestPoint_Pad_D1.0mm, symbol Connector:TestPoint
- added TP5: GND, TestPoint:TestPoint_Pad_D1.0mm, symbol Connector:TestPoint
- added TP6: VCC, TestPoint:TestPoint_Pad_D1.0mm, symbol Connector:TestPoint
- added U20: W25Q128JVS, Package_SO:SOIC-8_5.23x5.23mm_P1.27mm, symbol Memory_Flash:W25Q128JVS
Connections:
- net CONF_CLK: now also U20.6 (CLK)
- net CONF_IO0: now also U20.5 (DI(IO0))
- net CONF_IO1: now also U20.2 (DO(IO1))
- net CONF_IO2: now also U20.3 (IO2)
- net CONF_IO3: now also U20.7 (IO3)
- net CONF_M1: now also JP1.1 (A)
- net GND: now also C86.1, JP1.2 (B), TP5.1, U20.4 (GND)
- net TCK: now also TP4.1
- net TDI: now also TP1.1
- net TDO: now also TP2.1
- net TMS: now also TP3.1
- net VCC3_3: now also C86.2, R20.1, TP6.1, U20.8 (VCC)
- net ~{CONF_CS}: now also R20.2, U20.1 (~{CS})
- net UBUS_20: now reaches U7.M4 (IO_L1P_3)
- net UBUS_14: now reaches U7.M5 (IO_L2P_3)
- net UBUS_18: now reaches U7.N5 (IO_L49P_D3_2)
- net UBUS_12: now reaches U7.N6 (IO_L64N_D9_2)
- net UBUS_19: now reaches U7.N8 (IO_L29N_GCLK2_2)
- net UBUS_16: now reaches U7.P6 (IO_L47P_2)
- net UBUS_15: now reaches U7.P7 (IO_L31P_GCLK31_D14_2)
- net UBUS_17: now reaches U7.P8 (IO_L30P_GCLK1_D13_2)
- net UBUS_13: now reaches U7.R7 (IO_L32P_GCLK29_2)
- net UBUS_21: now reaches U7.R9 (IO_L23P_2)
- net UBUS_22: now reaches U7.T5 (IO_L48N_RDWR_B_VREF_2)
- no-connect marks 12 -> 1
Other:
- note added: "JTAG"
- note added: "Optional flash"

Commit message: revG
Connections:
- net ADC_BCK: now also U7.T7 (IO_L32N_GCLK28_2); no longer U7.T4 (IO_L63N_2)
- net ADC_LRCK: now also U7.T4 (IO_L63N_2); no longer U7.T7 (IO_L32N_GCLK28_2)
- net FT_CLK renamed VGA_R7
- net FT_DISP renamed MCU_IO4
- net MCU_SCK renamed VGA_R6
- net MIDI_CLK renamed UBUS_25
- net ~{ESP_BOOT} renamed UBUS_26
- net ~{ESP_RESET} renamed UBUS_27
- net ~{MIDI_RST} renamed UBUS_24

Commit message: rev.G2 WIP
Parts:
- removed C86: 100n, Capacitor_SMD:C_0603_1608Metric_Pad1.08x0.95mm_HandSolder, symbol Device:C
- removed JP1: Flashboot, Jumper:SolderJumper-2_P1.3mm_Open_RoundedPad1.0x1.5mm, symbol Jumper:Jumper_2_Open
- removed R20: 10k, Resistor_SMD:R_0603_1608Metric_Pad0.98x0.95mm_HandSolder, symbol Device:R
- removed U20: W25Q128JVS, Package_SO:SOIC-8_5.23x5.23mm_P1.27mm, symbol Memory_Flash:W25Q128JVS
- added TP10: IO0, TestPoint:TestPoint_Pad_D1.0mm, symbol Connector:TestPoint
- added TP11: IO2, TestPoint:TestPoint_Pad_D1.0mm, symbol Connector:TestPoint
- added TP12: IO3, TestPoint:TestPoint_Pad_D1.0mm, symbol Connector:TestPoint
- TP1, TP2, TP3, TP4, TP5, TP6: now left out of the parts list
Connections:
- net CONF_IO0: now also TP10.1
- net CONF_IO2: now also TP11.1
- net CONF_IO3: now also TP12.1
- net ~{CONF_CS} renamed ~{SDR_CS}
Other:
- note removed: "Optional flash"
