File: interfaces.kicad_sch (KiCad schematic)
At the start: 79 parts, among them J6 Tape In/Out, J7 Type-C right angle "flag" type, J8 Audio, J9 5V, U12 LM1117MP-3.3, U13 LM1117MP-1.2, U14 LM311, U15 SAM2695, U16 PCM1808PWR, U17 ESP-12E, U18 LM1117MP-3.3, U21 UDA1334ATS, Y3 12MHz

Commit message: rev.G2 WIP
Parts:
- removed C40, C41, C80: 10u, Capacitor_SMD:C_0603_1608Metric_Pad1.08x0.95mm_HandSolder, symbol Device:C
- removed C77, C78, C79, C92: 100n, Capacitor_SMD:C_0603_1608Metric_Pad1.08x0.95mm_HandSolder, symbol Device:C
- removed R71, R72: 220k, Resistor_SMD:R_0603_1608Metric_Pad0.98x0.95mm_HandSolder, symbol Device:R
- removed R73, R90: 100, Resistor_SMD:R_0603_1608Metric_Pad0.98x0.95mm_HandSolder, symbol Device:R
- removed U21: UDA1334ATS, Package_SO:SSOP-16_4.4x5.2mm_P0.65mm, symbol Audio:UDA1334ATS
- added C100, C98: 2n2, Capacitor_SMD:C_0603_1608Metric_Pad1.08x0.95mm_HandSolder, symbol Device:C
- added C101, C95, C97: 100n, Capacitor_SMD:C_0603_1608Metric_Pad1.08x0.95mm_HandSolder, symbol Device:C
- added C104, C105, C96, C99: 10u, Capacitor_SMD:C_0603_1608Metric_Pad1.08x0.95mm_HandSolder, symbol Device:C
- added C86: 2u2, Capacitor_SMD:C_0603_1608Metric_Pad1.08x0.95mm_HandSolder, symbol Device:C
- added R60: 1k, Resistor_SMD:R_0603_1608Metric_Pad0.98x0.95mm_HandSolder, symbol Device:R
- added R63, R64: 10k, Resistor_SMD:R_0603_1608Metric_Pad0.98x0.95mm_HandSolder, symbol Device:R
- added U25: PCM5102A, Package_SO:TSSOP-20_4.4x6.5mm_P0.65mm, symbol Audio:PCM5102A
Connections:
- net AUDIO_L: now also C104.1
- net AUDIO_R: now also C105.1
- net DAC_BCK: now also U25.13 (BCK)
- net DAC_DAT: now also U25.14 (DIN)
- net DAC_WS: now also U25.15 (LRCK)
- net GND: now also C100.1, C101.1, C95.2, C96.1, C97.1, C98.1, C99.1, U25.10 (DEMP), U25.11 (FLT), U25.12 (SCK), U25.16 (FMT), U25.19 (DGND), U25.3 (CPGND), U25.9 (AGND)
- net VCC3_3: now also C95.1, R60.1, U25.1 (CPVDD), U25.20 (DVDD), U25.8 (AVDD)
- new net: C101.2, C99.2, U25.18 (LDOO)
- new net: R60.2, U25.17 (XSMT)
- new net: C100.2, C105.2, R64.2
- new net: C96.2, C97.2, U25.5 (VNEG)
- new net: C86.2, U25.2 (CAPP)
- new net: C86.1, U25.4 (CAPM)
- new net: R63.1, U25.6 (OUTL)
- new net: R64.1, U25.7 (OUTR)
- new net: C104.2, C98.2, R63.2
Other:
- moved on the sheet: C75, C76, C81, C82, J8, R47, R48, R49, R52, R53, R54, R55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
