File: rp2040.kicad_sch (KiCad schematic)
At the start: 51 parts, among them J4 2x USB A, J5 2x USB A, U10 DS3231MZ, U2 LM1117MP-3.3, U3 W25Q128JVS, U4 RP2040, U8 FE1.1s, U9 24LC08B, Y1 12MHz, Y2 12MHz

Commit message: Updated revA: replaced resistors with IC for HDMI protection
Parts:
- renumbered C63 to C20, C20 to C21, C21 to C22, C22 to C23, J4 to J1, J5 to J2, R8 to R10, R75 to R11, R27 to R5, R28 to R6, R5 to R7, R6 to R8, R74 to R9, U2 to U1, U3 to U2, U4 to U3, U8 to U4, U9 to U5, U10 to U6

Commit message: Updated revB
Parts:
- added TP10: ADC0, TestPoint:TestPoint_Pad_D1.0mm, symbol Connector:TestPoint
- added TP11: ADC1, TestPoint:TestPoint_Pad_D1.0mm, symbol Connector:TestPoint
- added TP12: ADC2, TestPoint:TestPoint_Pad_D1.0mm, symbol Connector:TestPoint
- added TP13: ADC3, TestPoint:TestPoint_Pad_D1.0mm, symbol Connector:TestPoint
- added TP7: CLK, TestPoint:TestPoint_Pad_D1.0mm, symbol Connector:TestPoint
- added TP8: GND, TestPoint:TestPoint_Pad_D1.0mm, symbol Connector:TestPoint
- added TP9: IO, TestPoint:TestPoint_Pad_D1.0mm, symbol Connector:TestPoint
Connections:
- net GND: now also TP8.1
- net SWCLK: now also TP7.1
- net SWDIO: now also TP9.1
- net at U3.38 (GPIO26_ADC0): now also TP10.1
- net at U3.39 (GPIO27_ADC1): now also TP11.1
- net at U3.40 (GPIO28_ADC2): now also TP12.1
- net at U3.41 (GPIO29_ADC3): now also TP13.1
- no-connect marks 12 -> 8
Other:
- note added: "SWD"

Commit message: revF
Parts:
- added P4: I2C, Connector_PinHeader_1.27mm:PinHeader_1x04_P1.27mm_Vertical, symbol Connector_Generic:Conn_01x04
Connections:
- net GND: now also P4.4 (Pin_4)
- net I2C_SCL: now also P4.3 (Pin_3)
- net I2C_SDA: now also P4.2 (Pin_2)
- net VCC3_3: now also P4.1 (Pin_1)
Changed lines of the file:
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@@
   (title_block
     (title "Karabas-Mini")
-    (date "2024-04-17")
-    (rev "D")
+    (date "2024-05-25")
+    (rev "F")
   )
   (junction (at 226.06 87.63) (diameter 0) (color 0 0 0 0)
@@
     (stroke (width 0) (type default))
   )
+  (wire (pts (xy 269.24 64.77) (xy 271.78 64.77))
+    (stroke (width 0) (type default))
+  )
   (wire (pts (xy 231.14 92.71) (xy 210.82 92.71))
     (stroke (width 0) (type default))
@@
     (stroke (width 0) (type default))
   )
+  (wire (pts (xy 269.24 62.23) (xy 271.78 62.23))
+    (stroke (width 0) (type default))
+  )
   (wire (pts (xy 88.9 39.37) (xy 88.9 40.64))
     (stroke (width 0) (type default))
@@
     )
   )
+  (global_label "I2C_SDA" (shape bidirectional) (at 269.24 62.23 180) (fields_autoplaced)
+    (effects (font (size 1.27 1.27)) (justify right))
+    (property "Intersheetrefs" "${INTERSHEET_REFS}" (at 257.5235 62.23 0)
+      (effects (font (size 1.27 1.27)) (justify right) hide)
+    )
+  )
   (global_label "USBH_D+" (shape input) (at 208.28 106.68 180) (fields_autoplaced)
     (effects (font (size 1.27 1.27)) (justify right))
@@
     )
   )
+  (global_label "I2C_SCL" (shape bidirectional) (at 269.24 64.77 180) (fields_autoplaced)
+    (effects (font (size 1.27 1.27)) (justify right))
+    (property "Intersheetrefs" "${INTERSHEET_REFS}" (at 257.584 64.77 0)
+      (effects (font (size 1.27 1.27)) (justify right) hide)
+    )
+  )
   (global_label "I2C_SDA" (shape bidirectional) (at 245.11 55.88 0) (fields_autoplaced)
     (effects (font (size 1.27 1.27)) (justify left))
@@
     )
   )
+  (symbol (lib_id "Connector_Generic:Conn_01x04") (at 276.86 62.23 0) (unit 1)
+    (in_bom yes) (on_board yes) (dnp no) (fields_autoplaced)
+    (property "Reference" "P4" (at 279.4 62.23 0)
+      (effects (font (size 1.27 1.27)) (justify left))
+    )
+    (property "Value" "I2C" (at 279.4 64.77 0)
+      (effects (font (size 1.27 1.27)) (justify left))
+    )
+    (property "Footprint" "Connector_PinHeader_1.27mm:PinHeader_1x04_P1.27mm_Vertical" (at 276.86 62.23 0)
+      (effects (font (size 1.27 1.27)) hide)
+    )
+    (property "Datasheet" "~" (at 276.86 62.23 0)
+      (effects (font (size 1.27 1.27)) hide)
+    )
+    (pin "4")
+    (pin "1")
+    (pin "3")
+    (pin "2")
+    (instances
+      (project "karabas-mini"
+        (path "/3ea0d469-753b-4b31-8a3d-1341413bdcc8/aeb25ef9-b705-4fe0-b117-b7f20e33e486"
+          (reference "P4") (unit 1)
+        )
+      )
+    )
+  )
   (symbol (lib_id "power:GND") (at 278.13 156.21 0) (unit 1)
     (in_bom yes) (on_board yes) (dnp no)
@@
     )
   )
+  (symbol (lib_id "vcc33:VCC3_3") (at 271.78 59.69 0) (unit 1)
+    (in_bom yes) (on_board yes) (dnp no)
+    (property "Reference" "#PWR0110" (at 271.78 63.5 0)
+      (effects (font (size 1.27 1.27)) hide)
+    )
+    (property "Value" "VCC3_3" (at 270.51 55.88 0)
+      (effects (font (size 1.27 1.27)))
+    )
+    (property "Footprint" "" (at 271.78 59.69 0)
+      (effects (font (size 1.27 1.27)) hide)
+    )
+    (property "Datasheet" "" (at 271.78 59.69 0)
+      (effects (font (size 1.27 1.27)) hide)
+    )
+    (pin "1")
+    (instances
+      (project "karabas-mini"
+        (path "/3ea0d469-753b-4b31-8a3d-1341413bdcc8/aeb25ef9-b705-4fe0-b117-b7f20e33e486"
+          (reference "#PWR0110") (unit 1)
+        )
+      )
+    )
+  )
   (symbol (lib_id "Connector:USB_A_Stacked") (at 270.51 140.97 0) (mirror y) (unit 1)
     (in_bom yes) (on_board yes) (dnp no)
@@
         )
       )
+    )
+  )
+  (symbol (lib_id "power:GND") (at 271.78 67.31 0) (unit 1)
+    (in_bom yes) (on_board yes) (dnp no)
+    (property "Reference" "#PWR0111" (at 271.78 73.66 0)
+      (effects (font (size 1.27 1.27)) hide)
+    )
+    (property "Value" "GND" (at 271.907 71.7042 0)
+      (effects (font (size 1.27 1.27)))
+    )
+    (property "Footprint" "" (at 271.78 67.31 0)
+      (effects (font (size 1.27 1.27)) hide)
+    )
+    (property "Datasheet" "" (at 271.78 67.31 0)
+      (effects (font (size 1.27 1.27)) hide)
+    )
+    (pin "1")
+    (instances
+      (project "karabas-mini"
+        (path "/3ea0d469-753b-4b31-8a3d-1341413bdcc8/aeb25ef9-b705-4fe0-b117-b7f20e33e486"
+          (reference "#PWR0111") (unit 1)
+        )
+      )

Commit message: revG
Parts:
- removed TP10: ADC0, TestPoint:TestPoint_Pad_D1.0mm, symbol Connector:TestPoint
- removed TP11: ADC1, TestPoint:TestPoint_Pad_D1.0mm, symbol Connector:TestPoint
- removed TP12: ADC2, TestPoint:TestPoint_Pad_D1.0mm, symbol Connector:TestPoint
- removed TP13: ADC3, TestPoint:TestPoint_Pad_D1.0mm, symbol Connector:TestPoint
Connections:
- net MCU_IO4: now also U3.38 (GPIO26_ADC0); no longer U3.29 (GPIO18)
- net ~{MIDI_RST}: now reaches U3.40 (GPIO28_ADC2)
- net ~{FT_PD}: now reaches U3.39 (GPIO27_ADC1)
- net ~{ESP_RESET}: now reaches U3.41 (GPIO29_ADC3)
- new net MCU_IO5: U3.29 (GPIO18)

Commit message: rev.G2 WIP
Parts:
- TP7, TP8, TP9: now left out of the parts list
