File: vga.kicad_sch (KiCad schematic)
At the start: 19 parts, among them J2 HDMI_A_1.4, U5 FT812, Y3 8MHz

Commit message: Updated revA: replaced resistors with IC for HDMI protection
Parts:
- removed R10, R13, R14, R15, R16, R7: 270, Resistor_SMD:R_0603_1608Metric_Pad0.98x0.95mm_HandSolder, symbol Device:R
- added C83, C84, C85: 100n, Capacitor_SMD:C_0603_1608Metric_Pad1.08x0.95mm_HandSolder, symbol Device:C
- added R19: 10k, Resistor_SMD:R_0603_1608Metric_Pad0.98x0.95mm_HandSolder, symbol Device:R
- added U19: TPD12S016RKTR, footprints:IC_TPD12S016RKTR, symbol TPD12S016RKTR:TPD12S016RKTR
- R17, R18: value 270 -> 10k
- renumbered C28 to C38, C25 to C39, C23 to C40, C24 to C41, C27 to C42, C26 to C43, J2 to J3, R20 to R15, R19 to R16, U5 to U8
Connections:
- net D0N is gone; now on net HDMI_D0N: J3.9 (D0-)
- net D0P is gone; now on net HDMI_D0P: J3.7 (D0+)
- net D1N is gone; now on net HDMI_D1N: J3.6 (D1-)
- net D1P is gone; now on net HDMI_D1P: J3.4 (D1+)
- net D2N is gone; now on net HDMI_D2N: J3.3 (D2-)
- net D2P is gone; now on net HDMI_D2P: J3.1 (D2+)
- net GND: now also C83.1, C84.1, C85.2, U19.13 (GND), U19.18 (GND), U19.5 (GND)
- net HDMI_CKN: now also J3.12 (CK-), U19.14 (CLK-); no longer R18.1
- net HDMI_CKP: now also J3.10 (CK+), U19.15 (CLK+); no longer R17.1
- net HDMI_D0N: now also U19.16 (D0-)
- net HDMI_D0P: now also U19.17 (D0+)
- net HDMI_D1N: now also U19.19 (D1-)
- net HDMI_D1P: now also U19.20 (D1+)
- net HDMI_D2N: now also U19.21 (D2-)
- net HDMI_D2P: now also U19.22 (D2+)
- net VCC3_3: now also R17.2, R18.2, C84.2, R19.1, U19.11 (CT_HPD), U19.23 (VCCA), U19.4 (LS_OE)
- net CEC_B: now reaches J3.13 (CEC)
- net CEC_B: now also U19.6 (CEC_B)
- net SCL_B: now reaches J3.15 (SCL)
- net SCL_B: now also U19.7 (SCL_B)
- net SDA_B: now reaches J3.16 (SDA)
- net SDA_B: now also U19.8 (SDA_B)
- net HDMI_5V: now reaches J3.18 (+5V)
- net HDMI_5V: now also C85.1, U19.12 (5V_OUT)
- net HPD_B: now reaches J3.19 (HPD/HEAC-)
- net HPD_B: now also U19.9 (HPD_B)
- removed net CKN: J3.12 (CK-), R18.2
- removed net CKP: J3.10 (CK+), R17.2
- new net: R17.1, U19.1 (SCL_A)
- new net: R18.1, U19.2 (SDA_A)
- new net: R19.2, U19.3 (HPD_A)
- new net VCC: C83.2, U19.10 (VCC5V)
- no-connect marks 12 -> 11
Other:
- moved on the sheet: J3

Commit message: Updated revB
Parts:
- U8: footprint Package_DFN_QFN:QFN-56-1EP_7x7mm_P0.4mm_EP4x4mm -> Package_DFN_QFN:QFN-56-1EP_8x8mm_P0.5mm_EP5.9x5.9mm
Changed lines of the file:
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@@
   (title_block
     (title "Karabas-Mini")
-    (date "2024-02-20")
-    (rev "A")
+    (date "2024-02-23")
+    (rev "B")
   )
   (junction (at 77.47 62.23) (diameter 0) (color 0 0 0 0)
@@
       (effects (font (size 1.27 1.27)))
     )
-    (property "Footprint" "Package_DFN_QFN:QFN-56-1EP_7x7mm_P0.4mm_EP4x4mm" (at 105.41 147.32 0)
-      (effects (font (size 1.27 1.27)) hide)
-    )
+    (property "Footprint" "Package_DFN_QFN:QFN-56-1EP_8x8mm_P0.5mm_EP5.9x5.9mm" (at 105.41 147.32 0)
+      (effects (font (size 1.27 1.27)) hide)
+    )

Commit message: Fixed HDMI diff-pairs pinout, rev.C
Parts:
- added C87, C88, C89: 4n7, Capacitor_SMD:C_0603_1608Metric_Pad1.08x0.95mm_HandSolder, symbol Device:C
- added C90, C91: 10u, Capacitor_SMD:C_0603_1608Metric_Pad1.08x0.95mm_HandSolder, symbol Device:C
- added JP2: FT Audio L, Jumper:SolderJumper-2_P1.3mm_Open_RoundedPad1.0x1.5mm, symbol Jumper:Jumper_2_Open
- added JP3: FT Audio R, Jumper:SolderJumper-2_P1.3mm_Open_RoundedPad1.0x1.5mm, symbol Jumper:Jumper_2_Open
- added R21, R22, R23, R24, R56: 1k, Resistor_SMD:R_0603_1608Metric_Pad0.98x0.95mm_HandSolder, symbol Device:R
Connections:
- net FT_AUDIO: now also R21.1
- net GND: now also C87.2, C88.2, C89.2
- new net: C91.2, R56.1
- new net: JP3.1 (A), R56.2
- new net: C87.1, R21.2, R22.1
- new net: C89.1, C90.1, C91.1, R23.2
- new net: JP2.1 (A), R24.2
- new net: C90.2, R24.1
- new net: C88.1, R22.2, R23.1
- new net MIDI_L: JP2.2 (B)
- new net MIDI_R: JP3.2 (B)
Other:
- note added: "Optional analog audio capture DO NOT POPULATE"

Commit message: revG
Parts:
- removed C40, C41: 18pF, Capacitor_SMD:C_0603_1608Metric_Pad1.08x0.95mm_HandSolder, symbol Device:C
- removed JP2: FT Audio L, Jumper:SolderJumper-2_P1.3mm_Open_RoundedPad1.0x1.5mm, symbol Jumper:Jumper_2_Open
- removed JP3: FT Audio R, Jumper:SolderJumper-2_P1.3mm_Open_RoundedPad1.0x1.5mm, symbol Jumper:Jumper_2_Open
- removed Y3: 8MHz, Crystal:Crystal_SMD_3225-4Pin_3.2x2.5mm_HandSoldering, symbol Device:Crystal_GND24
- added D5: BAT54C, Package_TO_SOT_SMD:SOT-23, symbol Diode:BAT54C
Connections:
- net HDMI_5V: now also D5.3
- net MIDI_L: now also R24.2
- net MIDI_R: now also R56.2
- net VCC: now also D5.1
- net FT_CLK_X: now reaches U8.16 (X1)
- net FT_GPIO1: now reaches U8.10 (GPIO1(IO3))
- net FT_GPIO0: now reaches U8.9 (GPIO0(IO2))
- net FT_DISP: no longer names the net of U8.32 (DISP)
- no-connect marks 11 -> 12
Other:
- note added: "HDMI power (opt)"
- note removed: "Optional analog audio capture DO NOT POPULATE"
